Commit message: Controller Added

File: src/quadruped_robot/urdf/quadruped_robot.urdf.xacro (robot description, xacro)
@@ -1,6 +1,3 @@
 <?xml version="1.0"?>
-<!-- This URDF was automatically created by SolidWorks to URDF Exporter! Originally created by Stephen Brawner (brawner@gmail.com)
-     Commit Version: 1.6.0-4-g7f85cfe  Build Version: 1.6.7995.38578
-     For more information, please see http://wiki.ros.org/sw_urdf_exporter -->
 <robot name="quadruped_robot" xmlns:xacro="http://ros.org/wiki/xacro">
   <link
@@ -817,3 +814,110 @@
       xyz="0 0 0" />
   </joint>
+<gazebo>
+    <plugin filename="libgazebo_ros2_control.so" name="gazebo_ros2_control">
+        <parameters>$(find quadruped_robot)/config/control.yaml</parameters>
+    </plugin>
+</gazebo>
+<ros2_control name="GazeboSystem" type="system">
+ <hardware>
+     <plugin>gazebo_ros2_control/GazeboSystem</plugin>
+ </hardware>
+# Position Controller
+ <joint name="frs_joint">
+     <command_interface name="position">
+         <param name="min">-3.14</param>
+         <param name="max">3.14</param>
+     </command_interface>
+     <state_interface name="position"/>
+     <state_interface name="velocity"/>
+ </joint>
+  <joint name="fre_joint">
+     <command_interface name="position">
+         <param name="min">-3.14</param>
+         <param name="max">3.14</param>
+     </command_interface>
+     <state_interface name="position"/>
+     <state_interface name="velocity"/>
+ </joint>
+ <joint name="frw_joint">
+     <command_interface name="position">
+         <param name="min">-3.14</param>
+         <param name="max">3.14</param>
+     </command_interface>
+     <state_interface name="position"/>
+     <state_interface name="velocity"/>
+ </joint>
+  <joint name="rrs_joint">
+     <command_interface name="position">
+         <param name="min">-3.14</param>
+         <param name="max">3.14</param>
+     </command_interface>
+     <state_interface name="position"/>
+     <state_interface name="velocity"/>
+ </joint>
+ <joint name="rre_joint">
+     <command_interface name="position">
+         <param name="min">-3.14</param>
+         <param name="max">3.14</param>
+     </command_interface>
+     <state_interface name="position"/>
+     <state_interface name="velocity"/>
+ </joint>
+  <joint name="rrw_joint">
+     <command_interface name="position">
+         <param name="min">-3.14</param>
+         <param name="max">3.14</param>
+     </command_interface>
+     <state_interface name="position"/>
+     <state_interface name="velocity"/>
+ </joint>
+ <joint name="fls_joint">
+     <command_interface name="position">
+         <param name="min">-3.14</param>
+         <param name="max">3.14</param>
+     </command_interface>
+     <state_interface name="position"/>
+     <state_interface name="velocity"/>
+ </joint>
+  <joint name="fle_joint">
+     <command_interface name="position">
+         <param name="min">-3.14</param>
+         <param name="max">3.14</param>
+     </command_interface>
+     <state_interface name="position"/>
+     <state_interface name="velocity"/>
+ </joint>
+  <joint name="flw_joint">
+     <command_interface name="position">
+         <param name="min">-3.14</param>
+         <param name="max">3.14</param>
+     </command_interface>
+     <state_interface name="position"/>
+     <state_interface name="velocity"/>
+ </joint>
+  <joint name="rls_joint">
+     <command_interface name="position">
+         <param name="min">-3.14</param>
+         <param name="max">3.14</param>
+     </command_interface>
+     <state_interface name="position"/>
+     <state_interface name="velocity"/>
+ </joint>
+ <joint name="rle_joint">
+     <command_interface name="position">
+         <param name="min">-3.14</param>
+         <param name="max">3.14</param>
+     </command_interface>
+     <state_interface name="position"/>
+     <state_interface name="velocity"/>
+ </joint>
+  <joint name="rlw_joint">
+     <command_interface name="position">
+         <param name="min">-3.14</param>
+         <param name="max">3.14</param>
+     </command_interface>
+     <state_interface name="position"/>
+     <state_interface name="velocity"/>
+ </joint>
+ </ros2_control>
 </robot>

Commit message: Controller Updated

File: src/quadruped_robot/urdf/quadruped_robot.urdf.xacro (robot description, xacro)
@@ -814,110 +814,109 @@
       xyz="0 0 0" />
   </joint>
-<gazebo>
+  <gazebo>
     <plugin filename="libgazebo_ros2_control.so" name="gazebo_ros2_control">
-        <parameters>$(find quadruped_robot)/config/control.yaml</parameters>
+      <parameters>$(find quadruped_robot)/config/control.yaml</parameters>
     </plugin>
-</gazebo>
-<ros2_control name="GazeboSystem" type="system">
- <hardware>
-     <plugin>gazebo_ros2_control/GazeboSystem</plugin>
- </hardware>
-# Position Controller
- <joint name="frs_joint">
-     <command_interface name="position">
-         <param name="min">-3.14</param>
-         <param name="max">3.14</param>
-     </command_interface>
-     <state_interface name="position"/>
-     <state_interface name="velocity"/>
- </joint>
+  </gazebo>
+  <ros2_control name="GazeboSystem" type="system">
+    <hardware>
+      <plugin>gazebo_ros2_control/GazeboSystem</plugin>
+    </hardware> # Position Controller <joint
+      name="frs_joint">
+      <command_interface name="position">
+        <param name="min">-3.14</param>
+        <param name="max">3.14</param>
+      </command_interface>
+      <state_interface name="position" />
+      <state_interface name="velocity" />
+    </joint>
   <joint name="fre_joint">
-     <command_interface name="position">
-         <param name="min">-3.14</param>
-         <param name="max">3.14</param>
-     </command_interface>
-     <state_interface name="position"/>
-     <state_interface name="velocity"/>
- </joint>
+      <command_interface name="position">
+        <param name="min">-3.14</param>
+        <param name="max">3.14</param>
+      </command_interface>
+      <state_interface name="position" />
+      <state_interface name="velocity" />
+    </joint>
  <joint name="frw_joint">
-     <command_interface name="position">
-         <param name="min">-3.14</param>
-         <param name="max">3.14</param>
-     </command_interface>
-     <state_interface name="position"/>
-     <state_interface name="velocity"/>
- </joint>
+      <command_interface name="position">
+        <param name="min">-3.14</param>
+        <param name="max">3.14</param>
+      </command_interface>
+      <state_interface name="position" />
+      <state_interface name="velocity" />
+    </joint>
   <joint name="rrs_joint">
-     <command_interface name="position">
-         <param name="min">-3.14</param>
-         <param name="max">3.14</param>
-     </command_interface>
-     <state_interface name="position"/>
-     <state_interface name="velocity"/>
- </joint>
+      <command_interface name="position">
+        <param name="min">-3.14</param>
+        <param name="max">3.14</param>
+      </command_interface>
+      <state_interface name="position" />
+      <state_interface name="velocity" />
+    </joint>
  <joint name="rre_joint">
-     <command_interface name="position">
-         <param name="min">-3.14</param>
-         <param name="max">3.14</param>
-     </command_interface>
-     <state_interface name="position"/>
-     <state_interface name="velocity"/>
- </joint>
+      <command_interface name="position">
+        <param name="min">-3.14</param>
+        <param name="max">3.14</param>
+      </command_interface>
+      <state_interface name="position" />
+      <state_interface name="velocity" />
+    </joint>
   <joint name="rrw_joint">
-     <command_interface name="position">
-         <param name="min">-3.14</param>
-         <param name="max">3.14</param>
-     </command_interface>
-     <state_interface name="position"/>
-     <state_interface name="velocity"/>
- </joint>
+      <command_interface name="position">
+        <param name="min">-3.14</param>
+        <param name="max">3.14</param>
+      </command_interface>
+      <state_interface name="position" />
+      <state_interface name="velocity" />
+    </joint>
  <joint name="fls_joint">
-     <command_interface name="position">
-         <param name="min">-3.14</param>
-         <param name="max">3.14</param>
-     </command_interface>
-     <state_interface name="position"/>
-     <state_interface name="velocity"/>
- </joint>
+      <command_interface name="position">
+        <param name="min">-3.14</param>
+        <param name="max">3.14</param>
+      </command_interface>
+      <state_interface name="position" />
+      <state_interface name="velocity" />
+    </joint>
   <joint name="fle_joint">
-     <command_interface name="position">
-         <param name="min">-3.14</param>
-         <param name="max">3.14</param>
-     </command_interface>
-     <state_interface name="position"/>
-     <state_interface name="velocity"/>
- </joint>
+      <command_interface name="position">
+        <param name="min">-3.14</param>
+        <param name="max">3.14</param>
+      </command_interface>
+      <state_interface name="position" />
+      <state_interface name="velocity" />
+    </joint>
   <joint name="flw_joint">
-     <command_interface name="position">
-         <param name="min">-3.14</param>
-         <param name="max">3.14</param>
-     </command_interface>
-     <state_interface name="position"/>
-     <state_interface name="velocity"/>
- </joint>
+      <command_interface name="position">
+        <param name="min">-3.14</param>
+        <param name="max">3.14</param>
+      </command_interface>
+      <state_interface name="position" />
+      <state_interface name="velocity" />
+    </joint>
   <joint name="rls_joint">
-     <command_interface name="position">
-         <param name="min">-3.14</param>
-         <param name="max">3.14</param>
-     </command_interface>
-     <state_interface name="position"/>
-     <state_interface name="velocity"/>
- </joint>
+      <command_interface name="position">
+        <param name="min">-3.14</param>
+        <param name="max">3.14</param>
+      </command_interface>
+      <state_interface name="position" />
+      <state_interface name="velocity" />
+    </joint>
  <joint name="rle_joint">
-     <command_interface name="position">
-         <param name="min">-3.14</param>
-         <param name="max">3.14</param>
-     </command_interface>
-     <state_interface name="position"/>
-     <state_interface name="velocity"/>
- </joint>
+      <command_interface name="position">
+        <param name="min">-3.14</param>
+        <param name="max">3.14</param>
+      </command_interface>
+      <state_interface name="position" />
+      <state_interface name="velocity" />
+    </joint>
   <joint name="rlw_joint">
-     <command_interface name="position">
-         <param name="min">-3.14</param>
-         <param name="max">3.14</param>
-     </command_interface>
-     <state_interface name="position"/>
-     <state_interface name="velocity"/>
- </joint>
- </ros2_control>
+      <command_interface name="position">
+        <param name="min">-3.14</param>
+        <param name="max">3.14</param>
+      </command_interface>
+      <state_interface name="position" />
+      <state_interface name="velocity" />
+    </joint>
+  </ros2_control>
 </robot>

Commit message: added controller with inverse kinematics

File: src/quadruped_robot/urdf/quadruped_robot.urdf.xacro (robot description, xacro)
@@ -1,4 +1,10 @@
 <?xml version="1.0"?>
-<robot name="quadruped_robot" xmlns:xacro="http://ros.org/wiki/xacro">
+<robot
+  name="quadruped_robot" xmlns:xacro="http://ros.org/wiki/xacro">
+  <link name="dummy_link"></link> # Add this after base link <joint name="dummy_joint" type="fixed">
+    <origin rpy="0 0 0" xyz="0 0 0" />
+    <parent link="dummy_link" />
+    <child link="body_link" />
+  </joint>
   <link
     name="body_link">
@@ -8,12 +14,12 @@
         rpy="0 0 0" />
       <mass
-        value="0.377252605852233" />
-      <inertia
-        ixx="0.000418954363866351"
-        ixy="7.511988833675E-07"
-        ixz="4.09865880530585E-06"
-        iyy="0.000433125892291076"
-        iyz="1.41818186723719E-08"
-        izz="0.000626600145088028" />
+        value="2.8" />
+      <inertia
+        ixx="100"
+        ixy="0"
+        ixz="0"
+        iyy="100"
+        iyz="0"
+        izz="100" />
     </inertial>
     <visual>
@@ -48,12 +54,12 @@
         rpy="0 0 0" />
       <mass
-        value="0.0385204737997983" />
-      <inertia
-        ixx="8.71211945498261E-06"
-        ixy="4.10847903075371E-08"
-        ixz="-1.78152149761969E-10"
-        iyy="5.13274302177548E-06"
-        iyz="2.46917233525575E-07"
-        izz="7.80614050595697E-06" />
+        value="0.15" />
+      <inertia
+        ixx="100"
+        ixy="0"
+        ixz="0"
+        iyy="100"
+        iyz="0"
+        izz="100" />
     </inertial>
     <visual>
@@ -96,8 +102,8 @@
       lower="-1.04"
       upper="1.04"
-      effort="15"
-      velocity="0.1" />
-    <dynamics
-      friction="0.1" />
+      effort="20"
+      velocity="6" />
+    <dynamics damping="0.01"
+      friction="0.6" />
   </joint>
   <link
@@ -108,12 +114,12 @@
         rpy="0 0 0" />
       <mass
-        value="0.0887724177691983" />
-      <inertia
-        ixx="5.33826954697177E-05"
-        ixy="-4.01657420177436E-05"
-        ixz="2.23436712556012E-07"
-        iyy="5.54056136320405E-05"
-        iyz="1.34175995588459E-06"
-        izz="9.09432485780886E-05" />
+        value="0.15" />
+      <inertia
+        ixx="100"
+        ixy="0"
+        ixz="0"
+        iyy="100"
+        iyz="0"
+        izz="100" />
     </inertial>
     <visual>
@@ -152,12 +158,12 @@
       link="fre_link" />
     <axis
-      xyz="0 0 -1" />
+      xyz="0 0 1" />
     <limit
       lower="-1.57"
       upper="1.57"
-      effort="15"
-      velocity="0.1" />
-    <dynamics
-      friction="0.1" />
+      effort="20"
+      velocity="6" />
+    <dynamics damping="0.01"
+      friction="0.6" />
   </joint>
   <link
@@ -168,12 +174,12 @@
         rpy="0 0 0" />
       <mass
-        value="0.0364534542471395" />
-      <inertia
-        ixx="3.24424063682796E-05"
-        ixy="2.86763548564017E-05"
-        ixz="2.62022167693562E-06"
-        iyy="3.69606897466966E-05"
-        iyz="-2.37232854652557E-06"
-        izz="6.2793297163366E-05" />
+        value="0.15" />
+      <inertia
+        ixx="100"
+        ixy="0"
+        ixz="0"
+        iyy="100"
+        iyz="0"
+        izz="100" />
     </inertial>
     <visual>
@@ -199,4 +205,12 @@
           filename="package://quadruped_robot/meshes/frw_link.STL" />
       </geometry>
+      <surface>
+        <friction>
+          <ode>
+            <mu>0.1</mu>
+            <mu2>0.1</mu2>
+          </ode>
+        </friction>
+      </surface>
     </collision>
   </link>
@@ -212,12 +226,12 @@
       link="frw_link" />
     <axis
-      xyz="0 0 -1" />
+      xyz="0 0 1" />
     <limit
       lower="-1.57"
       upper="1.57"
-      effort="15"
-      velocity="0.1" />
-    <dynamics
-      friction="0.1" />
+      effort="20"
+      velocity="6" />
+    <dynamics damping="0.01"
+      friction="0.6" />
   </joint>
   <link
@@ -228,12 +242,12 @@
         rpy="0 0 0" />
       <mass
-        value="0.0385206604865966" />
-      <inertia
-        ixx="8.71226998638339E-06"
-        ixy="-4.115482434391E-08"
-        ixz="1.23274505723502E-10"
-        iyy="5.13285337559971E-06"
-        iyz="2.46844401583443E-07"
-        izz="7.80628697106784E-06" />
+        value="0.15" />
+      <inertia
+        ixx="100"
+        ixy="0"
+        ixz="0"
+        iyy="100"
+        iyz="0"
+        izz="100" />
     </inertial>
     <visual>
@@ -271,4 +285,192 @@
     <child
       link="rrs_link" />
+    <axis
+      xyz="0 0 1" />
+    <limit
+      lower="-1.04"
+      upper="1.04"
+      effort="20"
+      velocity="6" />
+    <dynamics damping="0.01"
+      friction="0.6" />
+  </joint>
+  <link
+    name="rre_link">
+    <inertial>
+      <origin
+        xyz="-0.0353949234320192 -0.0396843949308324 0.0318877499657951"
+        rpy="0 0 0" />
+      <mass
+        value="0.15" />
+      <inertia
+        ixx="100"
+        ixy="0"
+        ixz="0"
+        iyy="100"
+        iyz="0"
+        izz="100" />
+    </inertial>
+    <visual>
+      <origin
+        xyz="0 0 0"
+        rpy="0 0 0" />
+      <geometry>
+        <mesh
+          filename="package://quadruped_robot/meshes/rre_link.STL" />
+      </geometry>
+      <material
+        name="">
+        <color
+          rgba="0.2 0.2 0.2 1" />
+      </material>
+    </visual>
+    <collision>
+      <origin
+        xyz="0 0 0"
+        rpy="0 0 0" />
+      <geometry>
+        <mesh
+          filename="package://quadruped_robot/meshes/rre_link.STL" />
+      </geometry>
+    </collision>
+  </link>
+  <joint
+    name="rre_joint"
+    type="revolute">
+    <origin
+      xyz="-0.026 2.5092E-05 -0.0292"
+      rpy="0 -1.5708 0" />
+    <parent
+      link="rrs_link" />
+    <child
+      link="rre_link" />
+    <axis
+      xyz="0 0 1" />
+    <limit
+      lower="-1.57"
+      upper="1.57"
+      effort="20"
+      velocity="6" />
+    <dynamics damping="0.01"
+      friction="0.6" />
+  </joint>
+  <link
+    name="rrw_link">
+    <inertial>
+      <origin
+        xyz="0.0327282618505259 -0.0371355920751884 0.024575333341552"
+        rpy="0 0 0" />
+      <mass
+        value="0.15" />
+      <inertia
+        ixx="100"
+        ixy="0"
+        ixz="0"
+        iyy="100"
+        iyz="0"
+        izz="100" />
+    </inertial>
+    <visual>
+      <origin
+        xyz="0 0 0"
+        rpy="0 0 0" />
+      <geometry>
+        <mesh
+          filename="package://quadruped_robot/meshes/rrw_link.STL" />
+      </geometry>
+      <material
+        name="">
+        <color
+          rgba="0.2 0.2 0.2 1" />
+      </material>
+    </visual>
+    <collision>
+      <origin
+        xyz="0 0 0"
+        rpy="0 0 0" />
+      <geometry>
+        <mesh
+          filename="package://quadruped_robot/meshes/rrw_link.STL" />
+      </geometry>
+      <surface>
+        <friction>
+          <ode>
+            <mu>0.1</mu>
+            <mu2>0.1</mu2>
+          </ode>
+        </friction>
+      </surface>
+    </collision>
+  </link>
+  <joint
+    name="rrw_joint"
+    type="revolute">
+    <origin
+      xyz="-0.0674292551030644 -0.0855834232709074 0.0120000007629388"
+      rpy="0 0 0" />
+    <parent
+      link="rre_link" />
+    <child
+      link="rrw_link" />
+    <axis
+      xyz="0 0 1" />
+    <limit
+      lower="-1.57"
+      upper="1.57"
+      effort="20"
+      velocity="6" />
+    <dynamics damping="0.01"
+      friction="0.6" />
+  </joint>
+  <link
+    name="fls_link">
+    <inertial>
+      <origin
+        xyz="-0.0163097792199962 -0.00505189850993423 -0.0274848378346823"
+        rpy="0 0 0" />
+      <mass
+        value="0.15" />
+      <inertia
+        ixx="100"
+        ixy="0"
+        ixz="0"
+        iyy="100"
+        iyz="0"
+        izz="100" />
+    </inertial>
+    <visual>
+      <origin
+        xyz="0 0 0"
+        rpy="0 0 0" />
+      <geometry>
+        <mesh
+          filename="package://quadruped_robot/meshes/fls_link.STL" />
+      </geometry>
+      <material
+        name="">
+        <color
+          rgba="0.2 0.2 0.2 1" />
+      </material>
+    </visual>
+    <collision>
+      <origin
+        xyz="0 0 0"
+        rpy="0 0 0" />
+      <geometry>
+        <mesh
+          filename="package://quadruped_robot/meshes/fls_link.STL" />
+      </geometry>
+    </collision>
+  </link>
+  <joint
+    name="fls_joint"
+    type="revolute">
+    <origin
+      xyz="0.0692381468948904 0.041436948075885 0"
+      rpy="1.5707963267949 0 -1.5707963267949" />
+    <parent
+      link="body_link" />
+    <child
+      link="fls_link" />
     <axis
       xyz="0 0 -1" />
@@ -276,32 +478,32 @@
       lower="-1.04"
       upper="1.04"
-      effort="15"
-      velocity="0.1" />
-    <dynamics
-      friction="0.1" />
-  </joint>
-  <link
-    name="rre_link">
-    <inertial>
-      <origin
-        xyz="-0.0353949234320192 -0.0396843949308324 0.0318877499657951"
-        rpy="0 0 0" />
-      <mass
-        value="0.0887724191485841" />
-      <inertia
-        ixx="5.23102779505384E-05"
-        ixy="-4.01243985782808E-05"
-        ixz="2.41336508654976E-07"
-        iyy="5.64780329923361E-05"
-        iyz="1.33865580603777E-06"
-        izz="9.09432493810381E-05" />
-    </inertial>
-    <visual>
-      <origin
-        xyz="0 0 0"
-        rpy="0 0 0" />
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